Commit message: xacro files fixed

File: urdf/main.urdf.xacro (robot description, xacro)
@@ -31,10 +31,10 @@
 		<parent link="origin_link" />
 		<child link="base_link" />
-		<origin xyz="0 0 0.01905"/>
+		<origin xyz="0 0 0.020269"/>
 	</joint>
 	<xacro:rim_macro
 		name="left"
 		color="0.3 0 0"
-		xyz="-0.099 0.055 0.02"
+		xyz="-0.099 0.055 0.020269"
 		rpy="1.570796326794896 0 1.047197551196597"
 	/>
@@ -42,5 +42,5 @@
 		name="back"
 		color="0 0.3 0"
-		xyz="0 -0.11 0.02"
+		xyz="0 -0.11 0.020269"
 		rpy="1.570796326794896 0 3.141592653589793"
 	/>
@@ -48,5 +48,5 @@
 		name="right"
 		color="0 0 0.3"
-		xyz="0.099 0.055 0.02"
+		xyz="0.099 0.055 0.020269"
 		rpy="1.570796326794896 0 -1.047197551196597"
 	/>

File: urdf/rim.urdf.xacro (robot description, xacro)
@@ -8,12 +8,12 @@
 			<inertial>
 				<origin xyz="0 0 -0.000343"/>
-				<mass value="0.0083"/>
+				<mass value="0.083"/>
 				<inertia
-					ixx="0.2321e-04"
+					ixx="0.2198e-06"
 					ixy="0"
 					ixz="0"
-					iyy="0.2321e-04"
+					iyy="0.2198e-06"
 					iyz="0"
-					izz="0.3735e-04"/>
+					izz="0.3490e-06"/>
 			</inertial>
 			<visual>
@@ -44,5 +44,5 @@
 			parent="${name}"
 			name="upfront"
-			xyz="0 0.022 0"
+			xyz="0 0.022857 0"
 			rpy="-1.570796326794896 0 1.570796326794896"
 		/>
@@ -50,5 +50,5 @@
 			parent="${name}"
 			name="rightupfront"
-			xyz=" 0.02092 0.00679 0"
+			xyz=" 0.021738 0.007063 0"
 			rpy="-1.570796326794896 0 -2.82743"
 		/>
@@ -56,5 +56,5 @@
 			parent="${name}"
 			name="leftupfront"
-			xyz=" -0.02092 0.00679 0"
+			xyz=" -0.021738  0.007063 0"
 			rpy="-1.570796326794896 0 2.82743"
 		/>
@@ -62,5 +62,5 @@
 			parent="${name}"
 			name="rightdownfront"
-			xyz="0.01293 -0.01779 0"
+			xyz="0.013435 -0.018491 0"
 			rpy="-1.570796326794896 0 -0.959931"
 		/>
@@ -68,5 +68,5 @@
 			parent="${name}"
 			name="lefttdownfront"
-			xyz="-0.01293 -0.01779 0"
+			xyz="-0.013435 -0.018491 0"
 			rpy="-1.570796326794896 0 0.959931"
 		/>
@@ -75,5 +75,5 @@
 			parent="${name}"
 			name="upback"
-			xyz="0 -0.022 0.013"
+			xyz="0 -0.022857 0.013"
 			rpy="-1.570796326794896 0 1.570796326794896"
 		/>
@@ -81,5 +81,5 @@
 			parent="${name}"
 			name="rightupback"
-			xyz=" -0.02092 -0.00679 0.013"
+			xyz=" -0.021738 -0.007063 0.013"
 			rpy="-1.570796326794896 0 -2.82743"
 		/>
@@ -87,5 +87,5 @@
 			parent="${name}"
 			name="leftupback"
-			xyz=" 0.02092 -0.00679 0.013"
+			xyz=" 0.021738 -0.007063 0.013"
 			rpy="-1.570796326794896 0 2.82743"
 		/>
@@ -93,5 +93,5 @@
 			parent="${name}"
 			name="rightdownback"
-			xyz="-0.01293 0.01779 0.013"
+			xyz="-0.013435 0.018491 0.013"
 			rpy="-1.570796326794896 0 -0.959931"
 		/>
@@ -99,5 +99,5 @@
 			parent="${name}"
 			name="lefttdownback"
-			xyz="0.01293 0.01779 0.013"
+			xyz="0.013435 0.018491 0.013"
 			rpy="-1.570796326794896 0 0.959931"
 		/>

File: urdf/roller.urdf.xacro (robot description, xacro)
@@ -17,5 +17,5 @@
 			<visual>
 				<geometry>
-					<mesh filename="package://erobotica_omnibot/mesh/roller.stl"/>
+					<mesh filename="package://erobotica_omnibot/mesh/rolamento.stl"/>
 				</geometry>
 				<material name="roller_material">
@@ -25,5 +25,5 @@
 			<collision>
 				<geometry>
-					<mesh filename="package://erobotica_omnibot/mesh/roller.stl"/>
+					<mesh filename="package://erobotica_omnibot/mesh/rolamento.stl"/>
 				</geometry>
 			</collision>

Commit message: Add files via upload

File: urdf/main.urdf.xacro (robot description, xacro)
@@ -15,4 +15,5 @@
 		</inertial>
 	<visual>
+	<origin	xyz="0 0 0"  rpy="0 0 0" />
 		<geometry>
 			<mesh filename="package://erobotica_omnibot/mesh/chassi.stl"/>
@@ -23,4 +24,5 @@
 	</visual>
 	<collision>
+	<origin	xyz="0 0 0"  rpy="0 0 0" />
 		<geometry>
 			<mesh filename="package://erobotica_omnibot/mesh/chassi.stl"/>
@@ -31,10 +33,10 @@
 		<parent link="origin_link" />
 		<child link="base_link" />
-		<origin xyz="0 0 0.020269"/>
+		<origin xyz="0 0 0"/>
 	</joint>
 	<xacro:rim_macro
 		name="left"
 		color="0.3 0 0"
-		xyz="-0.0893842140 0.051606 0.020269"
+		xyz="-0.0893842140 0.051606 0.020272"
 		rpy="1.570796326794896 0 1.047197551196597"
 	/>
@@ -42,5 +44,5 @@
 		name="back"
 		color="0 0.3 0"
-		xyz="0 -0.103212  0.020269"
+		xyz="0 -0.103212  0.020272"
 		rpy="1.570796326794896 0 3.141592653589793"
 	/>
@@ -48,5 +50,5 @@
 		name="right"
 		color="0 0 0.3"
-		xyz="0.0893842140 0.051606 0.020269"
+		xyz="0.0893842140 0.051606 0.020272"
 		rpy="1.570796326794896 0 -1.047197551196597"
 	/>

File: urdf/rim.1aroda.xacro (robot description, xacro)
@@ -10,10 +10,10 @@
 				<mass value="0.083"/>
 				<inertia
-					ixx="0.1449e-04"
+					ixx="0.1846e-04"
 					ixy="0"
 					ixz="0"
-					iyy="0.1449e-04"
+					iyy="0.1846e-04"
 					iyz="0"
-					izz="0.2283e-04"/>
+					izz="0.3138e-04"/>
 			</inertial>
 			<visual>
@@ -38,5 +38,5 @@
 			<parent link="base_link" />
 			<child link="rim_${name}_link" />
-			<axis xyz="0 0 020269"/>
+			<axis xyz="0 0 1"/>
 			<origin xyz="${xyz}" rpy="${rpy}"/>
 		</joint>
@@ -44,5 +44,5 @@
 			parent="${name}"
 			name="upfront"
-			xyz="0 0.02406 0.006"
+			xyz="0 0.022857 0"
 			rpy="-1.570796326794896 0 1.570796326794896"
 		/>
@@ -50,5 +50,5 @@
 			parent="${name}"
 			name="rightupfront"
-			xyz=" 0.02288 0.00743 0.006"
+			xyz=" 0.021738 0.007063 0"
 			rpy="-1.570796326794896 0 -2.82743"
 		/>
@@ -56,5 +56,5 @@
 			parent="${name}"
 			name="leftupfront"
-			xyz=" -0.02288  0.00743 0.006"
+			xyz=" -0.021738  0.007063 0"
 			rpy="-1.570796326794896 0 2.82743"
 		/>
@@ -62,5 +62,5 @@
 			parent="${name}"
 			name="rightdownfront"
-			xyz="0.01414 -0.01947 0.006"
+			xyz="0.013435 -0.018491 0"
 			rpy="-1.570796326794896 0 -0.959931"
 		/>
@@ -68,5 +68,5 @@
 			parent="${name}"
 			name="lefttdownfront"
-			xyz="-0.01414 -0.01947 0.006"
+			xyz="-0.013435 -0.018491 0"
 			rpy="-1.570796326794896 0 0.959931"
 		/>
@@ -75,5 +75,5 @@
 			parent="${name}"
 			name="upback"
-			xyz="0 -0.02406 -0.006"
+			xyz="0 -0.022857 0.013"
 			rpy="-1.570796326794896 0 1.570796326794896"
 		/>
@@ -81,5 +81,5 @@
 			parent="${name}"
 			name="rightupback"
-			xyz=" -0.02288 -0.00743 -0.006"
+			xyz=" -0.021738 -0.007063 0.013"
 			rpy="-1.570796326794896 0 -2.82743"
 		/>
@@ -87,5 +87,5 @@
 			parent="${name}"
 			name="leftupback"
-			xyz=" 0.02288 -0.00743 -0.006"
+			xyz=" 0.021738 -0.007063 0.013"
 			rpy="-1.570796326794896 0 2.82743"
 		/>
@@ -93,5 +93,5 @@
 			parent="${name}"
 			name="rightdownback"
-			xyz="-0.01414 0.01947 -0.006"
+			xyz="-0.013435 0.018491 0.013"
 			rpy="-1.570796326794896 0 -0.959931"
 		/>
@@ -99,5 +99,5 @@
 			parent="${name}"
 			name="lefttdownback"
-			xyz="0.01414  0.01947 -0.006"
+			xyz="0.013435 0.018491 0.013"
 			rpy="-1.570796326794896 0 0.959931"
 		/>

File: urdf/roller.1orolamento.xacro (robot description, xacro)
@@ -8,10 +8,10 @@
 				<mass value="0.001"/>
 				<inertia
-					ixx="3.976186554728152e-08"
+					ixx="3.52707146475922e-08"
 					ixy="0"
 					ixz="0"
-					iyy="3.976186554728152e-08"
+					iyy="3.52714035128370e-08"
 					iyz="0"
-					izz="2.092071223656384e-08"/>
+					izz="1.29380165315134e-08"/>
 			</inertial>
 			<visual>
@@ -31,13 +31,4 @@
 	<gazebo reference="roller_${name}_rim_${parent}_link">
     		<material>Gazebo/Black</material>
-			<mu1 value="2.5" />
-			<mu2 value="2.5" />
-			<kp value="5000" />
-			<kd value="10" />
-						<!--<mu1 value="0.0"/>
-			<mu2 value="0.0"/>
-			<kp value="10000000.0" />
-			<kd value="1.0" />
-			<fdir1 value="0 0 1"/>-->
   	</gazebo>
 		<joint name="roller_${name}_rim_${parent}_joint" type="continuous">
@@ -46,5 +37,4 @@
 			<axis xyz="0 0 1"/>
 			<origin xyz="${xyz}" rpy="${rpy}"/>
-		<!--<dynamics damping="0.001"/>-->
 		</joint>
 	</xacro:macro>
